Commit message: deleted src, tried first implementation but has problems.
cartpole works --> so gymnasium pytorch etch are working

starting to build my own full environment

File: assets/URDF/aliengo.urdf (robot description, URDF)
Before this commit: robot aliengo, 31 links, 30 joints
Links:
- link FL_calf: geometry collision box size=0.25 0.0208 0.016; visual mesh filename=/home/rluser/RL_Dog/src/assets/MESHES/calf.dae scale=1 1 1
- link FL_hip: geometry collision cylinder length=0.0418 radius=0.046; visual mesh filename=/home/rluser/RL_Dog/src/assets/MESHES/hip.dae scale=1 1 1
- link FL_thigh: geometry collision box size=0.25 0.0374 0.043; visual mesh filename=/home/rluser/RL_Dog/src/assets/MESHES/thigh.dae scale=1 1 1
- link FR_calf: geometry collision box size=0.25 0.0208 0.016; visual mesh filename=/home/rluser/RL_Dog/src/assets/MESHES/calf.dae scale=1 1 1
- link FR_hip: geometry collision cylinder length=0.0418 radius=0.046; visual mesh filename=/home/rluser/RL_Dog/src/assets/MESHES/hip.dae scale=1 1 1
- link FR_thigh: geometry collision box size=0.25 0.0374 0.043; visual mesh filename=/home/rluser/RL_Dog/src/assets/MESHES/thigh_mirror.dae scale=1 1 1
- link RL_calf: geometry collision box size=0.25 0.0208 0.016; visual mesh filename=/home/rluser/RL_Dog/src/assets/MESHES/calf.dae scale=1 1 1
- link RL_hip: geometry collision cylinder length=0.0418 radius=0.046; visual mesh filename=/home/rluser/RL_Dog/src/assets/MESHES/hip.dae scale=1 1 1
- link RL_thigh: geometry collision box size=0.25 0.0374 0.043; visual mesh filename=/home/rluser/RL_Dog/src/assets/MESHES/thigh.dae scale=1 1 1
- link RR_calf: geometry collision box size=0.25 0.0208 0.016; visual mesh filename=/home/rluser/RL_Dog/src/assets/MESHES/calf.dae scale=1 1 1
- link RR_hip: geometry collision cylinder length=0.0418 radius=0.046; visual mesh filename=/home/rluser/RL_Dog/src/assets/MESHES/hip.dae scale=1 1 1
- link RR_thigh: geometry collision box size=0.25 0.0374 0.043; visual mesh filename=/home/rluser/RL_Dog/src/assets/MESHES/thigh_mirror.dae scale=1 1 1
- link trunk: geometry collision box size=0.647 0.15 0.112; visual mesh filename=/home/rluser/RL_Dog/src/assets/MESHES/trunk.dae scale=1 1 1

Commit message: done AnymalSimulation both rough and plain terrains

File: assets/URDF/aliengo.urdf (robot description, URDF)
Before this commit: robot aliengo, 31 links, 30 joints
Links:
- link FL_calf: geometry collision box size=0.25 0.0208 0.016; visual mesh filename=~/home/rluser/RL_Dog/src/assets/MESHES/calf.dae scale=1 1 1
- link FL_hip: geometry collision cylinder length=0.0418 radius=0.046; visual mesh filename=~/home/rluser/RL_Dog/src/assets/MESHES/hip.dae scale=1 1 1
- link FL_thigh: geometry collision box size=0.25 0.0374 0.043; visual mesh filename=~/home/rluser/RL_Dog/src/assets/MESHES/thigh.dae scale=1 1 1
- link FR_calf: geometry collision box size=0.25 0.0208 0.016; visual mesh filename=~/home/rluser/RL_Dog/src/assets/MESHES/calf.dae scale=1 1 1
- link FR_hip: geometry collision cylinder length=0.0418 radius=0.046; visual mesh filename=~/home/rluser/RL_Dog/src/assets/MESHES/hip.dae scale=1 1 1
- link FR_thigh: geometry collision box size=0.25 0.0374 0.043; visual mesh filename=~/home/rluser/RL_Dog/src/assets/MESHES/thigh_mirror.dae scale=1 1 1
- link RL_calf: geometry collision box size=0.25 0.0208 0.016; visual mesh filename=~/home/rluser/RL_Dog/src/assets/MESHES/calf.dae scale=1 1 1
- link RL_hip: geometry collision cylinder length=0.0418 radius=0.046; visual mesh filename=~/home/rluser/RL_Dog/src/assets/MESHES/hip.dae scale=1 1 1
- link RL_thigh: geometry collision box size=0.25 0.0374 0.043; visual mesh filename=~/home/rluser/RL_Dog/src/assets/MESHES/thigh.dae scale=1 1 1
- link RR_calf: geometry collision box size=0.25 0.0208 0.016; visual mesh filename=~/home/rluser/RL_Dog/src/assets/MESHES/calf.dae scale=1 1 1
- link RR_hip: geometry collision cylinder length=0.0418 radius=0.046; visual mesh filename=~/home/rluser/RL_Dog/src/assets/MESHES/hip.dae scale=1 1 1
- link RR_thigh: geometry collision box size=0.25 0.0374 0.043; visual mesh filename=~/home/rluser/RL_Dog/src/assets/MESHES/thigh_mirror.dae scale=1 1 1
- link trunk: geometry collision box size=0.647 0.15 0.112; visual mesh filename=~/home/rluser/RL_Dog/src/assets/MESHES/trunk.dae scale=1 1 1

Commit message: USD IS OK! is rendered ok in script 3 of tutorials
need to go on with train and env scripts

File: assets/URDF/aliengo.urdf (robot description, URDF)
Before this commit: robot aliengo, 31 links, 30 joints
Links:
- link FL_calf: geometry collision box size=0.25 0.0208 0.016; visual mesh filename=/home/rl_sim/RL_Dog/assets/MESHES/calf.dae scale=1 1 1
- link FL_hip: geometry collision cylinder length=0.0418 radius=0.046; visual mesh filename=/home/rl_sim/RL_Dog/assets/MESHES/hip.dae scale=1 1 1
- link FL_thigh: geometry collision box size=0.25 0.0374 0.043; visual mesh filename=/home/rl_sim/RL_Dog/assets/MESHES/thigh.dae scale=1 1 1
- link FR_calf: geometry collision box size=0.25 0.0208 0.016; visual mesh filename=/home/rl_sim/RL_Dog/assets/MESHES/calf.dae scale=1 1 1
- link FR_hip: geometry collision cylinder length=0.0418 radius=0.046; visual mesh filename=/home/rl_sim/RL_Dog/assets/MESHES/hip.dae scale=1 1 1
- link FR_thigh: geometry collision box size=0.25 0.0374 0.043; visual mesh filename=/home/rl_sim/RL_Dog/assets/MESHES/thigh_mirror.dae scale=1 1 1
- link RL_calf: geometry collision box size=0.25 0.0208 0.016; visual mesh filename=/home/rl_sim/RL_Dog/assets/MESHES/calf.dae scale=1 1 1
- link RL_hip: geometry collision cylinder length=0.0418 radius=0.046; visual mesh filename=/home/rl_sim/RL_Dog/assets/MESHES/hip.dae scale=1 1 1
- link RL_thigh: geometry collision box size=0.25 0.0374 0.043; visual mesh filename=/home/rl_sim/RL_Dog/assets/MESHES/thigh.dae scale=1 1 1
- link RR_calf: geometry collision box size=0.25 0.0208 0.016; visual mesh filename=/home/rl_sim/RL_Dog/assets/MESHES/calf.dae scale=1 1 1
- link RR_hip: geometry collision cylinder length=0.0418 radius=0.046; visual mesh filename=/home/rl_sim/RL_Dog/assets/MESHES/hip.dae scale=1 1 1
- link RR_thigh: geometry collision box size=0.25 0.0374 0.043; visual mesh filename=/home/rl_sim/RL_Dog/assets/MESHES/thigh_mirror.dae scale=1 1 1
- link trunk: geometry collision box size=0.647 0.15 0.112; visual mesh filename=/home/rl_sim/RL_Dog/assets/MESHES/trunk.dae scale=1 1 1
